File: pcb/pcjr-numpad.kicad_sch (KiCad schematic)
At the start: 54 parts, among them J1 USB_C_Receptacle_USB2.0_16P, J2 Conn_01x04, J3 Conn_01x02, Q1 AO3407, Q2 AO3407, SW1 SW_Push, SW10 SW_Push, SW11 SW_Push, SW12 SW_Push, SW13 SW_Push, SW14 SW_Push, SW15 SW_Push, SW16 SW_Push, SW17 SW_Push, SW2 SW_Push, SW3 SW_Push, SW4 SW_Push, SW5 SW_Push, SW6 SW_Push, SW7 SW_Push, SW8 SW_Push, SW9 SW_Push, U1 HOLYIOT-18010-NRF52840_Simple, U2 XC6220B331MR

Commit message: assign symbols with footprints
Parts:
- C1, C2, C3, C4, C5: footprint (none) -> pcjr-numpad-lib:C_0603
- D1, D10, D11, D12, D13, D14, D15, D16, D17, D2, D3, D4, D5, D6, D7, D8, D9: footprint Diode_SMD:D_SOD-123 -> pcjr-numpad-lib:D_SOD-123
- D18: footprint Diode_THT:D_DO-41_SOD81_P10.16mm_Horizontal -> pcjr-numpad-lib:D_SOD-123
- J1: footprint Package_DFN_QFN:WDFN-10-1EP_3x3mm_P0.5mm_EP1.8x2.5mm -> pcjr-numpad-lib:Connector_USB_C168688
- J2: footprint (none) -> pcjr-numpad-lib:Connector_THT_1x4_2.54mm
- J3: footprint (none) -> pcjr-numpad-lib:Connector_Battery_18650
- Q1: footprint (none) -> pcjr-numpad-lib:SOT-23-3
- Q2: footprint Package_DFN_QFN:AO_AOZ666xDI_DFN-8-1EP_3x3mm_P0.65mm_EP1.25x2.7mm -> pcjr-numpad-lib:SOT-23-3
- R1, R2: footprint Diode_THT:D_DO-41_SOD81_P10.16mm_Horizontal -> pcjr-numpad-lib:R_0603
- R3, R4, R5: footprint (none) -> pcjr-numpad-lib:R_0603
- SW1, SW10, SW11, SW12, SW13, SW14, SW17, SW2, SW3, SW4, SW5, SW6, SW7, SW9: footprint Button_Switch_SMD:Nidec_Copal_CAS-120A -> pcjr-numpad-lib:SW_Cherry_1.00U
- SW15, SW8: footprint Button_Switch_SMD:Nidec_Copal_CAS-120A -> pcjr-numpad-lib:SW_CHERRY_2.25U_Vertical
- SW16: footprint Button_Switch_SMD:Nidec_Copal_CAS-120A -> pcjr-numpad-lib:SW_Cherry_2.25U
- SW_PWR1: footprint Package_DFN_QFN:AO_AOZ666xDI_DFN-8-1EP_3x3mm_P0.65mm_EP1.25x2.7mm -> pcjr-numpad-lib:SW_MSK-12CO2
- SW_RST1: footprint Button_Switch_THT:SW_NKK_GW12LJP -> pcjr-numpad-lib:SW_K2-1187SQ
- U1: footprint (none) -> pcjr-numpad-lib:MCU_Holyiot-18010_mini
- U2: footprint Package_TO_SOT_SMD:SOT-23-5 -> pcjr-numpad-lib:SOT-23-5
Changed lines of the file:
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@@
 			)
 		)
-		(property "Footprint" ""
+		(property "Footprint" "pcjr-numpad-lib:R_0603"
 			(at 149.86 184.15 0)
 			(hide yes)
@@
 			)
 		)
-		(property "Footprint" "Button_Switch_SMD:Nidec_Copal_CAS-120A"
+		(property "Footprint" "pcjr-numpad-lib:SW_Cherry_1.00U"
 			(at 148.59 93.98 0)
 			(hide yes)
@@
 			)
 		)
-		(property "Footprint" "Button_Switch_SMD:Nidec_Copal_CAS-120A"
+		(property "Footprint" "pcjr-numpad-lib:SW_Cherry_1.00U"
 			(at 163.83 22.86 0)
 			(hide yes)
@@
 			)
 		)
-		(property "Footprint" ""
+		(property "Footprint" "pcjr-numpad-lib:C_0603"
 			(at 149.86 143.51 0)
 			(hide yes)
@@
 			)
 		)
-		(property "Footprint" "Diode_SMD:D_SOD-123"
+		(property "Footprint" "pcjr-numpad-lib:D_SOD-123"
 			(at 163.195 49.53 0)
 			(hide yes)
@@
 			)
 		)
-		(property "Footprint" "Diode_SMD:D_SOD-123"
+		(property "Footprint" "pcjr-numpad-lib:D_SOD-123"
 			(at 117.475 49.53 0)
 			(hide yes)
@@
 			)
 		)
-		(property "Footprint" "Button_Switch_THT:SW_NKK_GW12LJP"
+		(property "Footprint" "pcjr-numpad-lib:SW_K2-1187SQ"
 			(at 257.81 78.74 0)
 			(hide yes)
@@
 			)
 		)
-		(property "Footprint" "Button_Switch_SMD:Nidec_Copal_CAS-120A"
+		(property "Footprint" "pcjr-numpad-lib:SW_Cherry_1.00U"
 			(at 148.59 40.64 0)
 			(hide yes)
@@
 			)
 		)
-		(property "Footprint" "Diode_SMD:D_SOD-123"
+		(property "Footprint" "pcjr-numpad-lib:D_SOD-123"
 			(at 147.955 31.75 0)
 			(hide yes)
@@
 			)
 		)
-		(property "Footprint" "Package_DFN_QFN:AO_AOZ666xDI_DFN-8-1EP_3x3mm_P0.65mm_EP1.25x2.7mm"
+		(property "Footprint" "pcjr-numpad-lib:SOT-23-3"
 			(at 248.92 146.05 0)
 			(hide yes)
@@
 			)
 		)
-		(property "Footprint" ""
+		(property "Footprint" "pcjr-numpad-lib:Connector_THT_1x4_2.54mm"
 			(at 262.89 111.76 0)
 			(hide yes)
@@
 			)
 		)
-		(property "Footprint" ""
+		(property "Footprint" "pcjr-numpad-lib:MCU_Holyiot-18010_mini"
 			(at 54.61 58.42 0)
 			(hide yes)
@@
 			)
 		)
-		(property "Footprint" "Diode_THT:D_DO-41_SOD81_P10.16mm_Horizontal"
+		(property "Footprint" "pcjr-numpad-lib:D_SOD-123"
 			(at 26.67 172.085 0)
 			(hide yes)
@@
 			)
 		)
-		(property "Footprint" "Button_Switch_SMD:Nidec_Copal_CAS-120A"
+		(property "Footprint" "pcjr-numpad-lib:SW_Cherry_1.00U"
 			(at 133.35 22.86 0)
 			(hide yes)
@@
 			)
 		)
-		(property "Footprint" "Diode_SMD:D_SOD-123"
+		(property "Footprint" "pcjr-numpad-lib:D_SOD-123"
 			(at 117.475 67.31 0)
 			(hide yes)
@@
 			)
 		)
-		(property "Footprint" "Diode_THT:D_DO-41_SOD81_P10.16mm_Horizontal"
+		(property "Footprint" "pcjr-numpad-lib:R_0603"
 			(at 95.25 166.37 0)
 			(hide yes)
@@
 			)
 		)
-		(property "Footprint" "Package_TO_SOT_SMD:SOT-23-5"
+		(property "Footprint" "pcjr-numpad-lib:SOT-23-5"
 			(at 57.15 179.07 0)
 			(hide yes)
@@
 			)
 		)
-		(property "Footprint" "Button_Switch_SMD:Nidec_Copal_CAS-120A"
+		(property "Footprint" "pcjr-numpad-lib:SW_Cherry_1.00U"
 			(at 148.59 22.86 0)
 			(hide yes)
@@
 			)
 		)
-		(property "Footprint" ""
+		(property "Footprint" "pcjr-numpad-lib:C_0603"
 			(at 40.64 170.18 0)
 			(hide yes)
@@
 			)
 		)
-		(property "Footprint" ""
+		(property "Footprint" "pcjr-numpad-lib:C_0603"
 			(at 36.83 92.71 0)
 			(hide yes)
@@
 			)
 		)
-		(property "Footprint" "Package_DFN_QFN:WDFN-10-1EP_3x3mm_P0.5mm_EP1.8x2.5mm"
+		(property "Footprint" "pcjr-numpad-lib:Connector_USB_C168688"
 			(at 132.08 163.83 0)
 			(hide yes)
@@
 			)
 		)
-		(property "Footprint" ""
+		(property "Footprint" "pcjr-numpad-lib:SOT-23-3"
 			(at 31.75 162.56 0)
 			(hide yes)
@@
 			)
 		)
-		(property "Footprint" ""
+		(property "Footprint" "pcjr-numpad-lib:R_0603"
 			(at 95.25 177.8 0)
 			(hide yes)
@@
 			)
 		)
-		(property "Footprint" "Diode_SMD:D_SOD-123"
+		(property "Footprint" "pcjr-numpad-lib:D_SOD-123"
 			(at 147.955 102.87 0)
 			(hide yes)
@@
 			)
 		)
-		(property "Footprint" "Diode_SMD:D_SOD-123"
+		(property "Footprint" "pcjr-numpad-lib:D_SOD-123"
 			(at 117.475 31.75 0)
 			(hide yes)
@@
 			)
 		)
-		(property "Footprint" "Diode_THT:D_DO-41_SOD81_P10.16mm_Horizontal"
+		(property "Footprint" "pcjr-numpad-lib:R_0603"
 			(at 21.59 182.88 0)
 			(hide yes)
@@
 			)
 		)
-		(property "Footprint" "Diode_SMD:D_SOD-123"
+		(property "Footprint" "pcjr-numpad-lib:D_SOD-123"
 			(at 147.955 85.09 0)
 			(hide yes)
@@
 			)
 		)
-		(property "Footprint" "Button_Switch_SMD:Nidec_Copal_CAS-120A"
+		(property "Footprint" "pcjr-numpad-lib:SW_Cherry_1.00U"
 			(at 133.35 58.42 0)
 			(hide yes)
@@
 			)
 		)
-		(property "Footprint" "Diode_SMD:D_SOD-123"
+		(property "Footprint" "pcjr-numpad-lib:D_SOD-123"
 			(at 132.715 49.53 0)
 			(hide yes)
@@
 			)
 		)
-		(property "Footprint" ""
+		(property "Footprint" "pcjr-numpad-lib:Connector_Battery_18650"
 			(at 262.89 147.32 0)
 			(hide yes)
@@
 			)
 		)
-		(property "Footprint" "Package_DFN_QFN:AO_AOZ666xDI_DFN-8-1EP_3x3mm_P0.65mm_EP1.25x2.7mm"
+		(property "Footprint" "pcjr-numpad-lib:SW_MSK-12CO2"
 			(at 36.83 154.94 0)
 			(hide yes)
@@
 			)
 		)
-		(property "Footprint" "Button_Switch_SMD:Nidec_Copal_CAS-120A"
+		(property "Footprint" "pcjr-numpad-lib:SW_Cherry_1.00U"
 			(at 118.11 40.64 0)
 			(hide yes)
@@
 			)
 		)
-		(property "Footprint" ""
+		(property "Footprint" "pcjr-numpad-lib:C_0603"
 			(at 86.36 177.8 0)
 			(hide yes)
@@
 			)
 		)
-		(property "Footprint" "Button_Switch_SMD:Nidec_Copal_CAS-120A"
+		(property "Footprint" "pcjr-numpad-lib:SW_Cherry_1.00U"
 			(at 133.35 40.64 0)
 			(hide yes)
@@
 			)
 		)
-		(property "Footprint" "Diode_SMD:D_SOD-123"
+		(property "Footprint" "pcjr-numpad-lib:D_SOD-123"
 			(at 117.475 85.09 0)
 			(hide yes)
@@
 			)
 		)
-		(property "Footprint" "Button_Switch_SMD:Nidec_Copal_CAS-120A"
+		(property "Footprint" "pcjr-numpad-lib:SW_Cherry_2.25U"
 			(at 118.11 93.98 0)
 			(hide yes)
@@
 			)
 		)
-		(property "Footprint" ""
+		(property "Footprint" "pcjr-numpad-lib:C_0603"
 			(at 69.85 170.18 0)
 			(hide yes)
@@
 			)
 		)
-		(property "Footprint" "Button_Switch_SMD:Nidec_Copal_CAS-120A"
+		(property "Footprint" "pcjr-numpad-lib:SW_CHERRY_2.25U_Vertical"
 			(at 163.83 76.2 0)
 			(hide yes)
@@
 			)
 		)
-		(property "Footprint" "Diode_SMD:D_SOD-123"
+		(property "Footprint" "pcjr-numpad-lib:D_SOD-123"
 			(at 132.715 31.75 0)
 			(hide yes)
@@
 			)
 		)
-		(property "Footprint" "Button_Switch_SMD:Nidec_Copal_CAS-120A"
+		(property "Footprint" "pcjr-numpad-lib:SW_Cherry_1.00U"
 			(at 148.59 76.2 0)
 			(hide yes)
@@
 			)
 		)
-		(property "Footprint" "Button_Switch_SMD:Nidec_Copal_CAS-120A"
+		(property "Footprint" "pcjr-numpad-lib:SW_Cherry_1.00U"
 			(at 118.11 76.2 0)
 			(hide yes)
@@
 			)
 		)
-		(property "Footprint" "Button_Switch_SMD:Nidec_Copal_CAS-120A"
+		(property "Footprint" "pcjr-numpad-lib:SW_CHERRY_2.25U_Vertical"
 			(at 163.83 40.64 0)
 			(hide yes)
@@
 			)
 		)
-		(property "Footprint" "Button_Switch_SMD:Nidec_Copal_CAS-120A"
+		(property "Footprint" "pcjr-numpad-lib:SW_Cherry_1.00U"
 			(at 133.35 76.2 0)
 			(hide yes)
@@
 			)
 		)
-		(property "Footprint" "Diode_SMD:D_SOD-123"
+		(property "Footprint" "pcjr-numpad-lib:D_SOD-123"
 			(at 132.715 85.09 0)
 			(hide yes)
@@
 			)
 		)
-		(property "Footprint" ""
+		(property "Footprint" "pcjr-numpad-lib:R_0603"
 			(at 160.02 184.15 0)
 			(hide yes)
@@
 			)
 		)
-		(property "Footprint" "Diode_SMD:D_SOD-123"
+		(property "Footprint" "pcjr-numpad-lib:D_SOD-123"
 			(at 117.475 102.87 0)
 			(hide yes)
@@
 			)
 		)
-		(property "Footprint" "Button_Switch_SMD:Nidec_Copal_CAS-120A"
+		(property "Footprint" "pcjr-numpad-lib:SW_Cherry_1.00U"
 			(at 118.11 22.86 0)
 			(hide yes)
@@
 			)
 		)
-		(property "Footprint" "Diode_SMD:D_SOD-123"
+		(property "Footprint" "pcjr-numpad-lib:D_SOD-123"
 			(at 147.955 49.53 0)
 			(hide yes)
@@
 			)
 		)
-		(property "Footprint" "Button_Switch_SMD:Nidec_Copal_CAS-120A"
+		(property "Footprint" "pcjr-numpad-lib:SW_Cherry_1.00U"
 			(at 148.59 58.42 0)
 			(hide yes)
@@
 			)
 		)
-		(property "Footprint" "Button_Switch_SMD:Nidec_Copal_CAS-120A"
+		(property "Footprint" "pcjr-numpad-lib:SW_Cherry_1.00U"
 			(at 118.11 58.42 0)
 			(hide yes)
@@
 			)
 		)
-		(property "Footprint" "Diode_SMD:D_SOD-123"
+		(property "Footprint" "pcjr-numpad-lib:D_SOD-123"
 			(at 163.195 31.75 0)
 			(hide yes)
@@
 			)
 		)
-		(property "Footprint" "Diode_SMD:D_SOD-123"
+		(property "Footprint" "pcjr-numpad-lib:D_SOD-123"
 			(at 163.195 85.09 0)
 			(hide yes)
@@
 			)
 		)
-		(property "Footprint" "Diode_SMD:D_SOD-123"
+		(property "Footprint" "pcjr-numpad-lib:D_SOD-123"
 			(at 147.955 67.31 0)
 			(hide yes)
@@
 			)
 		)
-		(property "Footprint" "Diode_SMD:D_SOD-123"
+		(property "Footprint" "pcjr-numpad-lib:D_SOD-123"
 			(at 132.715 67.31 0)
 			(hide yes)

Commit message: reassign fixed footprints
Parts:
- SW15, SW8: footprint pcjr-numpad-lib:SW_CHERRY_2.25U_Vertical -> pcjr-numpad-lib:SW_Cherry_2.00U_Vertical
- SW16: footprint pcjr-numpad-lib:SW_Cherry_2.25U -> pcjr-numpad-lib:SW_Cherry_2.00U
Changed lines of the file:
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@@
 			)
 		)
-		(property "Footprint" "pcjr-numpad-lib:SW_Cherry_2.25U"
+		(property "Footprint" "pcjr-numpad-lib:SW_Cherry_2.00U"
 			(at 118.11 93.98 0)
 			(hide yes)
@@
 			)
 		)
-		(property "Footprint" "pcjr-numpad-lib:SW_CHERRY_2.25U_Vertical"
+		(property "Footprint" "pcjr-numpad-lib:SW_Cherry_2.00U_Vertical"
 			(at 163.83 76.2 0)
 			(hide yes)
@@
 			)
 		)
-		(property "Footprint" "pcjr-numpad-lib:SW_CHERRY_2.25U_Vertical"
+		(property "Footprint" "pcjr-numpad-lib:SW_Cherry_2.00U_Vertical"
 			(at 163.83 40.64 0)
 			(hide yes)
